File: electrical/pcb/uno_hat/uno_hat_dev.kicad_pcb (KiCad board)
At the start: 2 copper layers, 155 x 58.1 mm, 98 parts, among them J1 Conn_01x08_MountingPin, J2 Conn_01x08_MountingPin, Q1 NMOS, Q10 NMOS, Q11 NMOS, Q12 NMOS, Q13 NMOS, Q14 PMOS, Q15 PMOS, Q16 PMOS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

Commit message: Add files via upload
Connections:
- J1 pad 5: /DOT5 -> /DOT7
- J1 pad 7: /DOT7 -> /DOT5
Routing:
- net GND: track 111.4 -> 287.3 mm, vias 25 -> 36
- net GNDA: track 29.3 -> 185.9 mm, vias 4 -> 5
- net /UP4: track 9.77 -> 110.9 mm
- net /DOT5: track 0.00 -> 65.1 mm, vias 0 -> 1
- net /DOT1: track 0.00 -> 64.7 mm, vias 0 -> 1
- net /DOT2: track 0.00 -> 48.6 mm, vias 0 -> 1
- net /DOT6: track 0.00 -> 47.0 mm, vias 0 -> 1
- net /DOT3: track 0.00 -> 32.8 mm, vias 0 -> 1
- net /DOT4: track 0.00 -> 27.8 mm, vias 0 -> 1
- net /DOT7: track 0.00 -> 26.0 mm, vias 0 -> 1
- net /DOT8: track 0.00 -> 7.62 mm
- net /DOWN3: track 71.4 -> 70.4 mm
- net /+450V: track 168.6 -> 169.4 mm
- net /UP3: track 122.1 -> 122.8 mm
