File: electrical/pcb/uno_hat/uno_hat_dev.kicad_sch (KiCad schematic)
At the start: 2 parts, among them U1 LM5185QPWPRQ1

Commit message: Add files via upload
Parts:
- removed MOSFET1: STL90N6F7, POWERFLAT_5X6_C_STM, symbol 2026-03-06_23-43-22:STL90N6F7
- removed U1: LM5185QPWPRQ1, PWP0014G-IPC_A, symbol 2026-02-07_14-23-52:LM5185QPWPRQ1
- added A1: Arduino_UNO_R3, Module:Arduino_UNO_R3, symbol MCU_Module:Arduino_UNO_R3
- added C13: 100p, Resistor_SMD:R_0805_2012Metric, symbol Device:C
- added C14, C17: 250U, Capacitor_THT:CP_Radial_Tantal_D8.0mm_P2.50mm, symbol Device:C
- added C15, Cvcc2: 4.7uF, Resistor_SMD:R_0805_2012Metric, symbol Device:C
- added C16: 22p, Resistor_SMD:R_0805_2012Metric, symbol Device:C
- added C18: 820pF, Resistor_SMD:R_0805_2012Metric, symbol Device:C
- added C19: 10pF, Resistor_SMD:R_0805_2012Metric, symbol Device:C
- added Css2: 100nF, Resistor_SMD:R_0805_2012Metric, symbol Device:C
- added D1, D2, D3, D4, D5, D6, D7, D8: 1N47xxA, Diode_THT:D_DO-41_SOD81_P10.16mm_Horizontal, symbol Diode:1N47xxA
- added D10, D11, D12, D13, D14, D15, D16, D17, D18, D19, D20, D21, D22, D23, D24, D9: LED, LED_SMD:LED_0805_2012Metric, symbol Device:LED
- added D29: 500mV, Diode_THT:D_A-405_P12.70mm_Horizontal, symbol Device:D
- added J1, J2: Conn_01x08_MountingPin, Connector_FFC-FPC:Amphenol_F32Q-1A7x1-11008_1x08-1MP_P0.5mm_Horizontal, symbol Connector_Generic_MountingPin:Conn_01x08_MountingPin
- added Q1, Q10, Q11, Q12, Q13, Q4, Q6, Q8: NMOS, Package_TO_SOT_THT:TO-92_Inline, symbol Simulation_SPICE:NMOS
- added Q14, Q15, Q16, Q17, Q2, Q5, Q7, Q9: PMOS, Package_TO_SOT_THT:TO-92_Inline, symbol Simulation_SPICE:PMOS
- added Q20: NMOS, Package_TO_SOT_THT:TO-220-3_Vertical, symbol Simulation_SPICE:NMOS
- added Q3: NPN, Package_TO_SOT_THT:TO-92_Inline, symbol Simulation_SPICE:NPN
- added R1, R13, R14, R15, R16, R4, R6, R8: 10K, Resistor_THT:R_Axial_DIN0207_L6.3mm_D2.5mm_P7.62mm_Horizontal, symbol Device:R
- added R10, R11, R12, R2, R3, R5, R7, R9: 10M, Resistor_THT:R_Axial_DIN0207_L6.3mm_D2.5mm_P7.62mm_Horizontal, symbol Device:R
- added R17, R18, R19, R20, R21, R22, R23, R24, R25, R26, R27, R28, R29, R30, R31, R32: 330, Resistor_SMD:R_0805_2012Metric, symbol Device:R
- added R42, R46: 10kΩ, Resistor_SMD:R_0805_2012Metric, symbol Device:R
- added R43: 10k, Resistor_SMD:R_0805_2012Metric, symbol Device:R
- added R44: 100Ω, Resistor_SMD:R_0805_2012Metric, symbol Device:R
- added R45: 1k54, Resistor_SMD:R_0805_2012Metric, symbol Device:R
- added R47: 100, Resistor_SMD:R_0805_2012Metric, symbol Device:R
- added R48: R_Shunt, Resistor_SMD:R_Shunt_Ohmite_LVK24, symbol Device:R_Shunt
- added Rcs2: 0.1Ω, Resistor_SMD:R_0805_2012Metric, symbol Device:R
- added T2: Transformer_1P_1S, Connector_PinSocket_2.54mm:PinSocket_1x04_P2.54mm_Vertical, symbol Device:Transformer_1P_1S
- added U5: LM5185QPWPRQ1, Package_SO:Texas_HTSSOP-14-1EP_4.4x5mm_P0.65mm_EP3.4x5mm_Mask3.155x3.255mm, symbol 2026-02-07_14-23-52:LM5185QPWPRQ1
- added U6: INA219AxD, Package_SO:SOIC-8_3.9x4.9mm_P1.27mm, symbol Sensor_Energy:INA219AxD
Connections:
- new net: D6.2 (A), Q15.2 (G), R10.2, R14.2
- new net: Q10.1 (D), R9.1
- new net: D5.2 (A), Q14.2 (G), R13.2, R9.2
- new net: C13.1, R44.1, U5.9 (CS)
- new net: Q20.3 (S), R44.2, Rcs2.2
- new net: D2.2 (A), Q5.2 (G), R3.2, R4.2
- new net: D21.2 (A), R29.1
- new net: D1.2 (A), Q2.2 (G), R1.2, R2.2
- new net: D13.2 (A), R21.1
- new net: D19.2 (A), R27.1
- new net: D18.2 (A), R26.1
- new net: D22.2 (A), R30.1
- new net: Q11.1 (D), R10.1
- new net: D15.2 (A), R23.1
- new net: Q20.1 (D), R43.2, T2.2 (AB)
- new net: D29.2 (A), R47.1, T2.3 (SA)
- new net: D12.2 (A), R20.1
- new net: D16.2 (A), R24.1
- new net: Q1.1 (D), R2.1
- new net: D3.2 (A), Q7.2 (G), R5.2, R6.2
- new net: Q12.1 (D), R11.1
- new net: D24.2 (A), R32.1
- new net: D14.2 (A), R22.1
- new net: Css2.1, U5.6 (SS)
- new net: D20.2 (A), R28.1
- new net: D8.2 (A), Q17.2 (G), R12.2, R16.2
- new net: Q4.1 (D), R3.1
- new net: D9.2 (A), R17.1
- new net: Q8.1 (D), R7.1
- new net: Q20.2 (G), U5.11 (GATE)
- new net: D7.2 (A), Q16.2 (G), R11.2, R15.2
- new net: D23.2 (A), R31.1
- new net: D4.2 (A), Q9.2 (G), R7.2, R8.2
- new net: D17.2 (A), R25.1
- new net: Q13.1 (D), R12.1
- new net: Q6.1 (D), R5.1
- new net: Cvcc2.1, U5.10 (VCC)
- new net: R43.1, U5.13 (FB)
- new net: R42.2, U5.4 (RSET)
- new net: C16.1, R47.2
- new net: C18.1, R45.2
- new net: D10.2 (A), R18.1
- new net: D11.2 (A), R19.1
- new net +12V: C14.1, C17.1, R46.2, T2.1 (AA), U5.14 (VIN)
- new net +12V+: A1.8 (VIN), R48.2, R48.3, U6.7 (IN-), U6.8 (IN+)
- new net +450V: C15.1, C16.2, D1.1 (K), D2.1 (K), D29.1 (K), D3.1 (K), D4.1 (K), D5.1 (K), D6.1 (K), D7.1 (K), D8.1 (K), Q14.1 (D), Q15.1 (D), Q16.1 (D), Q17.1 (D), Q2.1 (D), Q5.1 (D), Q7.1 (D), Q9.1 (D), R1.1, R13.1, R14.1, R15.1, R16.1, R4.1, R6.1, R8.1
- new net +5VP: A1.5 (+5V), U6.5 (VS)
- new net COMP: C19.1, R45.1, U5.7 (COMP)
- new net DOT1: J1.1 (Pin_1), Q14.3 (S)
- new net DOT2: J1.2 (Pin_2), Q2.3 (S)
- new net DOT3: J1.3 (Pin_3), Q15.3 (S)
- new net DOT4: J1.4 (Pin_4), Q5.3 (S)
- new net DOT5: J1.5 (Pin_5), Q16.3 (S)
- new net DOT6: J1.6 (Pin_6), Q7.3 (S)
- new net DOT7: J1.7 (Pin_7), Q17.3 (S)
- new net DOT8: J1.8 (Pin_8), Q9.3 (S)
- new net DOWN1: A1.16 (D1/TX), R25.2
- new net DOWN2: A1.24 (D9), R26.2
- new net DOWN3: A1.10 (A1), A1.17 (D2), R27.2
- new net DOWN4: A1.11 (A2), R28.2
- new net DOWN5: A1.27 (D12), R29.2
- new net DOWN6: A1.23 (D8), R30.2
- new net DOWN7: A1.21 (D6), R31.2
- new net DOWN8: A1.19 (D4), R32.2
- new net EN: Q3.1 (C), R46.1, U5.1 (EN)
- new net GND: A1.29 (GND), A1.6 (GND), A1.7 (GND), C14.2, C15.2, C17.2, D10.1 (K), D11.1 (K), D12.1 (K), D13.1 (K), D14.1 (K), D15.1 (K), D16.1 (K), D17.1 (K), D18.1 (K), D19.1 (K), D20.1 (K), D21.1 (K), D22.1 (K), D23.1 (K), D24.1 (K), D9.1 (K), Q1.3 (S), Q10.3 (S), Q11.3 (S), Q12.3 (S), Q13.3 (S), Q3.3 (E), Q4.3 (S), Q6.3 (S), Q8.3 (S), T2.4 (SB), U6.1 (A1), U6.2 (A0), U6.6 (GND)
- new net GNDA: C13.2, C18.2, C19.2, Css2.2, Cvcc2.2, J2.1 (Pin_1), J2.2 (Pin_2), J2.3 (Pin_3), J2.4 (Pin_4), J2.5 (Pin_5), J2.6 (Pin_6), J2.7 (Pin_7), J2.8 (Pin_8), R42.1, Rcs2.1, U5.15 (EP), U5.5 (AGND), U5.8 (PGND)
- new net PWR_EN: A1.9 (A0), Q3.2 (B)
- new net SCL: A1.32 (SCL/A5), U6.4 (SCL)
- new net SDA: A1.31 (SDA/A4), U6.3 (SDA)
- new net UP1: A1.15 (D0/RX), Q10.2 (G), R17.2
- new net UP2: A1.25 (D10), Q1.2 (G), R18.2
- new net UP3: A1.18 (D3), Q11.2 (G), R19.2
- new net UP4: Q4.2 (G), R20.2
- new net UP5: A1.28 (D13), Q12.2 (G), R21.2
- new net UP6: A1.26 (D11), Q6.2 (G), R22.2
- new net UP7: A1.22 (D7), Q13.2 (G), R23.2
- new net UP8: A1.20 (D5), Q8.2 (G), R24.2
Other:
- note added: "CSD19534KCS"
- note added: "Leakage L: 4.04e-6 Lp (uH):202.00 NS1-NP: 4.00"

Commit message: Add files via upload
Connections:
- net DOT5: now also J1.7 (Pin_7); no longer J1.5 (Pin_5)
- net DOT7: now also J1.5 (Pin_5); no longer J1.7 (Pin_7)
Changed lines of the file:
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@@
 		)
 	)
-	(label "DOT7"
+	(label "DOT5"
 		(at 96.52 189.23 0)
 		(effects
@@
 		)
 	)
-	(label "DOT5"
+	(label "DOT7"
 		(at 96.52 184.15 0)
 		(effects
