File: electrical/pcb/demo_board/demo_board/demo_board.kicad_sch (KiCad schematic)
At the start: 9 parts, among them J5 Conn_01x02_Socket, J6 Conn_01x02_Socket, J7 Conn_01x06_Socket, J8 Conn_01x06_Pin, U1 74HC595, U2 74HC595, U3 74HC595, U4 SN74LV4T125

Commit message: Updated layout and board shape determined
Parts:
- R49: footprint Resistor_THT:R_Axial_DIN0207_L6.3mm_D2.5mm_P7.62mm_Horizontal -> Resistor_SMD:R_0603_1608Metric
- U1, U2, U3: footprint Package_DIP:DIP-16_W7.62mm -> Package_SO:SOIC-16W_5.3x10.2mm_P1.27mm
Changed lines of the file:
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@@
 			)
 		)
-		(property "Footprint" "Package_DIP:DIP-16_W7.62mm"
+		(property "Footprint" "Package_SO:SOIC-16W_5.3x10.2mm_P1.27mm"
 			(at 170.18 128.27 0)
 			(effects
@@
 			)
 		)
-		(property "Footprint" "Package_DIP:DIP-16_W7.62mm"
+		(property "Footprint" "Package_SO:SOIC-16W_5.3x10.2mm_P1.27mm"
 			(at 170.18 41.91 0)
 			(effects
@@
 			)
 		)
-		(property "Footprint" "Package_DIP:DIP-16_W7.62mm"
+		(property "Footprint" "Package_SO:SOIC-16W_5.3x10.2mm_P1.27mm"
 			(at 170.18 85.09 0)
 			(effects
@@
 			)
 		)
-		(property "Footprint" "Resistor_THT:R_Axial_DIN0207_L6.3mm_D2.5mm_P7.62mm_Horizontal"
+		(property "Footprint" "Resistor_SMD:R_0603_1608Metric"
 			(at 154.178 173.99 90)
 			(effects

Commit message: placement done
Connections:
- net DIN: now also J7.1 (Pin_1); no longer J8.1 (Pin_1)
- net DOUT: now also J8.1 (Pin_1); no longer J7.1 (Pin_1)
- net OE: now also J8.4 (Pin_4); no longer J7.4 (Pin_4)
- net OE_IN: now also J7.4 (Pin_4); no longer J8.4 (Pin_4)
- net RCLK: now also J8.3 (Pin_3); no longer J7.3 (Pin_3)
- net RCLK_IN: now also J7.3 (Pin_3); no longer J8.3 (Pin_3)
- net SRCLK: now also J8.2 (Pin_2); no longer J7.2 (Pin_2)
- net SRCLK_IN: now also J7.2 (Pin_2); no longer J8.2 (Pin_2)
Other:
- moved on the sheet: J7, J8
Changed lines of the file:
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@@
 	(symbol
 		(lib_id "Connector:Conn_01x06_Socket")
-		(at 59.69 140.97 0)
+		(at 29.21 118.11 0)
+		(mirror y)
 		(unit 1)
 		(exclude_from_sim no)
@@
 		(on_board yes)
 		(dnp no)
-		(fields_autoplaced yes)
 		(property "Reference" "J7"
-			(at 60.96 140.9699 0)
+			(at 27.94 118.1099 0)
 			(effects
 				(font
@@
 		)
 		(property "Value" "Conn_01x06_Socket"
-			(at 60.96 143.5099 0)
+			(at 27.94 120.6499 0)
 			(effects
 				(font
@@
 		)
 		(property "Footprint" "Connector_PinSocket_2.54mm:PinSocket_2x03_P2.54mm_Horizontal"
+			(at 29.21 118.11 0)
+			(effects
+				(font
+					(size 1.27 1.27)
+				)
+				(hide yes)
+			)
+		)
+		(property "Datasheet" "~"
+			(at 29.21 118.11 0)
+			(effects
+				(font
+					(size 1.27 1.27)
+				)
+				(hide yes)
+			)
+		)
+		(property "Description" "Generic connector, single row, 01x06, script generated"
+			(at 29.21 118.11 0)
+			(effects
+				(font
+					(size 1.27 1.27)
+				)
+				(hide yes)
+			)
+		)
+		(pin "3"
+		)
+		(pin "4"
+		)
+		(pin "1"
+		)
+		(pin "2"
+		)
+		(pin "5"
+		)
+		(pin "6"
+		)
+		(instances
+			(project "demo_board"
+				(path "/23e003c8-bfa5-4ac4-b719-34dc5a23b231"
+					(reference "J7")
+					(unit 1)
+				)
+			)
+		)
+	)
+	(symbol
+		(lib_id "Connector:Conn_01x06_Pin")
+		(at 59.69 140.97 0)
+		(mirror y)
+		(unit 1)
+		(exclude_from_sim no)
+		(in_bom yes)
+		(on_board yes)
+		(dnp no)
+		(property "Reference" "J8"
+			(at 59.055 130.81 0)
+			(effects
+				(font
+					(size 1.27 1.27)
+				)
+			)
+		)
+		(property "Value" "Conn_01x06_Pin"
+			(at 59.055 133.35 0)
+			(effects
+				(font
+					(size 1.27 1.27)
+				)
+			)
+		)
+		(property "Footprint" "Connector_PinHeader_2.54mm:PinHeader_2x03_P2.54mm_Horizontal"
 			(at 59.69 140.97 0)
 			(effects
@@
 		(pin "3"
 		)
-		(pin "4"
-		)
-		(pin "1"
-		)
-		(pin "2"
-		)
-		(pin "5"
-		)
-		(pin "6"
-		)
-		(instances
-			(project ""
-				(path "/23e003c8-bfa5-4ac4-b719-34dc5a23b231"
-					(reference "J7")
-					(unit 1)
-				)
-			)
-		)
-	)
-	(symbol
-		(lib_id "Connector:Conn_01x06_Pin")
-		(at 29.21 118.11 0)
-		(unit 1)
-		(exclude_from_sim no)
-		(in_bom yes)
-		(on_board yes)
-		(dnp no)
-		(fields_autoplaced yes)
-		(property "Reference" "J8"
-			(at 29.845 107.95 0)
-			(effects
-				(font
-					(size 1.27 1.27)
-				)
-			)
-		)
-		(property "Value" "Conn_01x06_Pin"
-			(at 29.845 110.49 0)
-			(effects
-				(font
-					(size 1.27 1.27)
-				)
-			)
-		)
-		(property "Footprint" "Connector_PinHeader_2.54mm:PinHeader_2x03_P2.54mm_Horizontal"
-			(at 29.21 118.11 0)
-			(effects
-				(font
-					(size 1.27 1.27)
-				)
-				(hide yes)
-			)
-		)
-		(property "Datasheet" "~"
-			(at 29.21 118.11 0)
-			(effects
-				(font
-					(size 1.27 1.27)
-				)
-				(hide yes)
-			)
-		)
-		(property "Description" "Generic connector, single row, 01x06, script generated"
-			(at 29.21 118.11 0)
-			(effects
-				(font
-					(size 1.27 1.27)
-				)
-				(hide yes)
-			)
-		)
-		(pin "3"
-		)
 		(pin "6"
 		)
@@
 		)
 		(instances
-			(project ""
+			(project "demo_board"
 				(path "/23e003c8-bfa5-4ac4-b719-34dc5a23b231"
 					(reference "J8")

Commit message: initial layout of dev
Changed lines of the file:
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@@
+		)
+	)
+	(global_label "+450V"
+		(shape input)
+		(at 27.94 173.99 90)
+		(fields_autoplaced yes)
+		(effects
+			(font
+				(size 1.27 1.27)
+			)
+			(justify left)
+		)
+		(property "Intersheetrefs" "${INTERSHEET_REFS}"
+			(at 27.94 164.7153 90)
+			(effects
+				(font
+					(size 1.27 1.27)
+				)
+				(justify left)
+				(hide yes)
+			)
 		)
 	)
@@
 				(hide yes)
 			)
+		)
+	)
+	(global_label "+450V"
+		(shape input)
+		(at 55.88 173.99 90)
+		(fields_autoplaced yes)
+		(effects
+			(font
+				(size 1.27 1.27)
+			)
+			(justify left)
+		)
+		(property "Intersheetrefs" "${INTERSHEET_REFS}"
+			(at 55.88 164.7153 90)
+			(effects
+				(font
+					(size 1.27 1.27)
+				)
+				(justify left)
+				(hide yes)
+			)
