File: electrical/pcb/demo_board/demo_board/dotdriver.kicad_sch (KiCad schematic)
At the start: 32 parts, among them J1 Conn_01x06_Socket, J2 Conn_01x06_Socket, Q1 NMOS, Q10 NMOS, Q11 NMOS, Q12 NMOS, Q14 PMOS, Q15 PMOS, Q16 PMOS, Q2 PMOS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

Commit message: Updated layout and board shape determined
Parts:
- D1, D2, D3, D5, D6, D7: value 1N47xxA -> BZT52C9V1-7-F; footprint Diode_THT:D_DO-41_SOD81_P10.16mm_Horizontal -> Diode_SMD:D_SOD-123
- Q1, Q10, Q11, Q12, Q14, Q15, Q16, Q2, Q4, Q5, Q6, Q7: footprint Package_TO_SOT_THT:TO-92_Inline -> Package_TO_SOT_SMD:SOT-89-3
- R1, R10, R11, R13, R14, R15, R2, R3, R4, R5, R6, R9: footprint Resistor_THT:R_Axial_DIN0207_L6.3mm_D2.5mm_P7.62mm_Horizontal -> Resistor_SMD:R_0603_1608Metric
Changed lines of the file:
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@@
 			)
 		)
-		(property "Footprint" "Resistor_THT:R_Axial_DIN0207_L6.3mm_D2.5mm_P7.62mm_Horizontal"
+		(property "Footprint" "Resistor_SMD:R_0603_1608Metric"
 			(at 82.042 52.07 90)
 			(effects
@@
 			)
 		)
-		(property "Footprint" "Resistor_THT:R_Axial_DIN0207_L6.3mm_D2.5mm_P7.62mm_Horizontal"
+		(property "Footprint" "Resistor_SMD:R_0603_1608Metric"
 			(at 76.2 32.258 90)
 			(effects
@@
 			)
 		)
-		(property "Footprint" "Resistor_THT:R_Axial_DIN0207_L6.3mm_D2.5mm_P7.62mm_Horizontal"
+		(property "Footprint" "Resistor_SMD:R_0603_1608Metric"
 			(at 156.972 52.07 90)
 			(effects
@@
 			)
 		)
-		(property "Footprint" "Package_TO_SOT_THT:TO-92_Inline"
+		(property "Footprint" "Package_TO_SOT_SMD:SOT-89-3"
 			(at 184.15 27.94 0)
 			(effects
@@
 			)
 		)
-		(property "Footprint" "Package_TO_SOT_THT:TO-92_Inline"
+		(property "Footprint" "Package_TO_SOT_SMD:SOT-89-3"
 			(at 74.93 58.42 0)
 			(effects
@@
 			)
 		)
-		(property "Footprint" "Resistor_THT:R_Axial_DIN0207_L6.3mm_D2.5mm_P7.62mm_Horizontal"
+		(property "Footprint" "Resistor_SMD:R_0603_1608Metric"
 			(at 151.13 32.258 90)
 			(effects
@@
 			)
 		)
-		(property "Footprint" "Package_TO_SOT_THT:TO-92_Inline"
+		(property "Footprint" "Package_TO_SOT_SMD:SOT-89-3"
 			(at 184.15 78.74 0)
 			(effects
@@
 			)
 		)
-		(property "Value" "1N47xxA"
+		(property "Value" "BZT52C9V1-7-F"
 			(at 170.18 78.7399 90)
 			(effects
@@
 			)
 		)
-		(property "Footprint" "Diode_THT:D_DO-41_SOD81_P10.16mm_Horizontal"
+		(property "Footprint" "Diode_SMD:D_SOD-123"
 			(at 163.195 77.47 0)
 			(effects
@@
 			)
 		)
-		(property "Datasheet" "https://www.vishay.com/docs/85816/1n4728a.pdf"
+		(property "Datasheet" "https://www.diodes.com/assets/Datasheets/ds18004.pdf"
 			(at 167.64 77.47 0)
 			(effects
@@
 			)
 		)
-		(property "Footprint" "Resistor_THT:R_Axial_DIN0207_L6.3mm_D2.5mm_P7.62mm_Horizontal"
+		(property "Footprint" "Resistor_SMD:R_0603_1608Metric"
 			(at 82.042 26.67 90)
 			(effects
@@
 			)
 		)
-		(property "Footprint" "Package_TO_SOT_THT:TO-92_Inline"
+		(property "Footprint" "Package_TO_SOT_SMD:SOT-89-3"
 			(at 74.93 83.82 0)
 			(effects
@@
 			)
 		)
-		(property "Footprint" "Package_TO_SOT_THT:TO-92_Inline"
+		(property "Footprint" "Package_TO_SOT_SMD:SOT-89-3"
 			(at 149.86 58.42 0)
 			(effects
@@
 			)
 		)
-		(property "Footprint" "Resistor_THT:R_Axial_DIN0207_L6.3mm_D2.5mm_P7.62mm_Horizontal"
+		(property "Footprint" "Resistor_SMD:R_0603_1608Metric"
 			(at 156.972 26.67 90)
 			(effects
@@
 			)
 		)
-		(property "Footprint" "Package_TO_SOT_THT:TO-92_Inline"
+		(property "Footprint" "Package_TO_SOT_SMD:SOT-89-3"
 			(at 149.86 33.02 0)
 			(effects
@@
 			)
 		)
-		(property "Footprint" "Resistor_THT:R_Axial_DIN0207_L6.3mm_D2.5mm_P7.62mm_Horizontal"
+		(property "Footprint" "Resistor_SMD:R_0603_1608Metric"
 			(at 76.2 83.058 90)
 			(effects
@@
 			)
 		)
-		(property "Footprint" "Package_TO_SOT_THT:TO-92_Inline"
+		(property "Footprint" "Package_TO_SOT_SMD:SOT-89-3"
 			(at 74.93 33.02 0)
 			(effects
@@
 			)
 		)
-		(property "Value" "1N47xxA"
+		(property "Value" "BZT52C9V1-7-F"
 			(at 95.25 53.3399 90)
 			(effects
@@
 			)
 		)
-		(property "Footprint" "Diode_THT:D_DO-41_SOD81_P10.16mm_Horizontal"
+		(property "Footprint" "Diode_SMD:D_SOD-123"
 			(at 88.265 52.07 0)
 			(effects
@@
 			)
 		)
-		(property "Datasheet" "https://www.vishay.com/docs/85816/1n4728a.pdf"
+		(property "Datasheet" "https://www.diodes.com/assets/Datasheets/ds18004.pdf"
 			(at 92.71 52.07 0)
 			(effects
@@
 			)
 		)
-		(property "Footprint" "Package_TO_SOT_THT:TO-92_Inline"
+		(property "Footprint" "Package_TO_SOT_SMD:SOT-89-3"
 			(at 149.86 83.82 0)
 			(effects
@@
 			)
 		)
-		(property "Value" "1N47xxA"
+		(property "Value" "BZT52C9V1-7-F"
 			(at 95.25 78.7399 90)
 			(effects
@@
 			)
 		)
-		(property "Footprint" "Diode_THT:D_DO-41_SOD81_P10.16mm_Horizontal"
+		(property "Footprint" "Diode_SMD:D_SOD-123"
 			(at 88.265 77.47 0)
 			(effects
@@
 			)
 		)
-		(property "Datasheet" "https://www.vishay.com/docs/85816/1n4728a.pdf"
+		(property "Datasheet" "https://www.diodes.com/assets/Datasheets/ds18004.pdf"
 			(at 92.71 77.47 0)
 			(effects
@@
 			)
 		)
-		(property "Value" "1N47xxA"
+		(property "Value" "BZT52C9V1-7-F"
 			(at 170.18 53.3399 90)
 			(effects
@@
 			)
 		)
-		(property "Footprint" "Diode_THT:D_DO-41_SOD81_P10.16mm_Horizontal"
+		(property "Footprint" "Diode_SMD:D_SOD-123"
 			(at 163.195 52.07 0)
 			(effects
@@
 			)
 		)
-		(property "Datasheet" "https://www.vishay.com/docs/85816/1n4728a.pdf"
+		(property "Datasheet" "https://www.diodes.com/assets/Datasheets/ds18004.pdf"
 			(at 167.64 52.07 0)
 			(effects
@@
 			)
 		)
-		(property "Footprint" "Package_TO_SOT_THT:TO-92_Inline"
+		(property "Footprint" "Package_TO_SOT_SMD:SOT-89-3"
 			(at 109.22 78.74 0)
 			(effects
@@
 			)
 		)
-		(property "Footprint" "Resistor_THT:R_Axial_DIN0207_L6.3mm_D2.5mm_P7.62mm_Horizontal"
+		(property "Footprint" "Resistor_SMD:R_0603_1608Metric"
 			(at 82.042 77.47 90)
 			(effects
@@
 			)
 		)
-		(property "Footprint" "Package_TO_SOT_THT:TO-92_Inline"
+		(property "Footprint" "Package_TO_SOT_SMD:SOT-89-3"
 			(at 109.22 53.34 0)
 			(effects
@@
 			)
 		)
-		(property "Footprint" "Resistor_THT:R_Axial_DIN0207_L6.3mm_D2.5mm_P7.62mm_Horizontal"
+		(property "Footprint" "Resistor_SMD:R_0603_1608Metric"
 			(at 151.13 83.058 90)
 			(effects
@@
 			)
 		)
-		(property "Footprint" "Resistor_THT:R_Axial_DIN0207_L6.3mm_D2.5mm_P7.62mm_Horizontal"
+		(property "Footprint" "Resistor_SMD:R_0603_1608Metric"
 			(at 151.13 57.658 90)
 			(effects
@@
 			)
 		)
-		(property "Footprint" "Package_TO_SOT_THT:TO-92_Inline"
+		(property "Footprint" "Package_TO_SOT_SMD:SOT-89-3"
 			(at 184.15 53.34 0)
 			(effects
@@
 			)
 		)
-		(property "Footprint" "Package_TO_SOT_THT:TO-92_Inline"
+		(property "Footprint" "Package_TO_SOT_SMD:SOT-89-3"
 			(at 109.22 27.94 0)
 			(effects
@@
 			)
 		)
-		(property "Footprint" "Resistor_THT:R_Axial_DIN0207_L6.3mm_D2.5mm_P7.62mm_Horizontal"
+		(property "Footprint" "Resistor_SMD:R_0603_1608Metric"
 			(at 76.2 57.658 90)
 			(effects
@@
 			)
 		)
-		(property "Value" "1N47xxA"
+		(property "Value" "BZT52C9V1-7-F"
 			(at 170.18 27.9399 90)
 			(effects
@@
 			)
 		)
-		(property "Footprint" "Diode_THT:D_DO-41_SOD81_P10.16mm_Horizontal"
+		(property "Footprint" "Diode_SMD:D_SOD-123"
 			(at 163.195 26.67 0)
 			(effects
@@
 			)
 		)
-		(property "Datasheet" "https://www.vishay.com/docs/85816/1n4728a.pdf"
+		(property "Datasheet" "https://www.diodes.com/assets/Datasheets/ds18004.pdf"
 			(at 167.64 26.67 0)
 			(effects
@@
 			)
 		)
-		(property "Footprint" "Resistor_THT:R_Axial_DIN0207_L6.3mm_D2.5mm_P7.62mm_Horizontal"
+		(property "Footprint" "Resistor_SMD:R_0603_1608Metric"
 			(at 156.972 77.47 90)
 			(effects
@@
 			)
 		)
-		(property "Value" "1N47xxA"
+		(property "Value" "BZT52C9V1-7-F"
 			(at 95.25 27.9399 90)
 			(effects
@@
 			)
 		)
-		(property "Footprint" "Diode_THT:D_DO-41_SOD81_P10.16mm_Horizontal"
+		(property "Footprint" "Diode_SMD:D_SOD-123"
 			(at 88.265 26.67 0)
 			(effects
@@
 			)
 		)
-		(property "Datasheet" "https://www.vishay.com/docs/85816/1n4728a.pdf"
+		(property "Datasheet" "https://www.diodes.com/assets/Datasheets/ds18004.pdf"
 			(at 92.71 26.67 0)
 			(effects

Commit message: initial layout of dev
Changed lines of the file:
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@@
+		)
+	)
+	(global_label "+450V"
+		(shape input)
+		(at 106.68 22.86 0)
+		(fields_autoplaced yes)
+		(effects
+			(font
+				(size 1.27 1.27)
+			)
+			(justify left)
+		)
+		(property "Intersheetrefs" "${INTERSHEET_REFS}"
+			(at 115.9547 22.86 0)
+			(effects
+				(font
+					(size 1.27 1.27)
+				)
+				(justify left)
+				(hide yes)
+			)
 		)
 	)

Commit message: layout finished
Parts:
- added R50, R54, R58, R62, R66, R70: 1K, Resistor_SMD:R_0603_1608Metric, symbol Device:R
Connections:
- net GND: now also R50.2, R54.2, R58.2, R62.2, R66.2, R70.2
- net UP1: now also R50.1
- net UP2: now also R62.1
- net UP3: now also R54.1
- net UP4: now also R66.1
- net UP5: now also R58.1
- net UP6: now also R70.1
