File: electrical/pcb/demo_board/demo_board/demo_board.kicad_pcb (KiCad board)
At the start: 2 copper layers, 137 parts, among them J0 Conn_01x06_Socket, J1 Conn_01x06_Socket, J10 Conn_01x06_Socket, J11 Conn_01x06_Socket, J2 Conn_01x06_Socket, J3 Conn_01x06_Socket, J4 Conn_01x06_Socket, J5 Conn_01x02_Socket, J6 Conn_01x02_Socket, J7 Conn_01x06_Socket, J8 Conn_01x06_Pin, J9 Conn_01x06_Socket, Q1 NMOS, Q10 NMOS, Q11 NMOS, Q12 NMOS, Q13 PMOS, Q14 PMOS, Q15 PMOS, Q16 PMOS, Q17 PMOS, Q18 PMOS, Q19 NMOS, Q2 PMOS, Q20 NMOS, Q21 NMOS, Q22 PMOS, Q23 PMOS, Q24 PMOS, Q25 NMOS, Q26 NMOS, Q27 NMOS, Q28 PMOS, Q29 PMOS, Q3 NMOS, Q30 PMOS, Q31 NMOS, Q32 NMOS, Q33 NMOS, Q34 PMOS, Q35 PMOS, Q36 PMOS, Q37 NMOS, Q38 NMOS, Q39 NMOS, Q4 NMOS, Q40 PMOS, Q41 PMOS, Q42 PMOS, Q43 NMOS, Q44 NMOS, Q45 NMOS, Q46 PMOS, Q47 PMOS, Q48 PMOS, Q5 PMOS, Q6 NMOS, Q7 PMOS, Q8 NMOS, Q9 NMOS, U1 74HC595, U2 74HC595, U3 74HC595, U4 SN74LV4T125

Commit message: Updated layout and board shape determined
Parts:
- added D13: BZT52C9V1-7-F, Diode_SMD:D_SOD-123, F.Cu at (58.1, 94.8)
- added D13: BZT52C9V1-7-F, Diode_SMD:D_SOD-123, F.Cu at (88.9, 94.8)
- added D13: BZT52C9V1-7-F, Diode_SMD:D_SOD-123, F.Cu at (42.7, 94.8)
- added D14: BZT52C9V1-7-F, Diode_SMD:D_SOD-123, F.Cu at (94.0, 95.0)
- added D14: BZT52C9V1-7-F, Diode_SMD:D_SOD-123, F.Cu at (63.2, 95.0)
- added D14: BZT52C9V1-7-F, Diode_SMD:D_SOD-123, F.Cu at (47.8, 95.0)
- added D15: BZT52C9V1-7-F, Diode_SMD:D_SOD-123, F.Cu at (99.2, 95.0)
- added D15: BZT52C9V1-7-F, Diode_SMD:D_SOD-123, F.Cu at (53.0, 95.0)
- added D15: BZT52C9V1-7-F, Diode_SMD:D_SOD-123, F.Cu at (68.4, 95.0)
- added D16: BZT52C9V1-7-F, Diode_SMD:D_SOD-123, F.Cu at (86.4, 118.9)
- added D16: BZT52C9V1-7-F, Diode_SMD:D_SOD-123, F.Cu at (55.7, 118.9)
- added D16: BZT52C9V1-7-F, Diode_SMD:D_SOD-123, F.Cu at (40.2, 118.9)
- added D17: BZT52C9V1-7-F, Diode_SMD:D_SOD-123, F.Cu at (45.4, 118.9)
- added D17: BZT52C9V1-7-F, Diode_SMD:D_SOD-123, F.Cu at (60.8, 118.9)
- added D17: BZT52C9V1-7-F, Diode_SMD:D_SOD-123, F.Cu at (91.6, 118.9)
- added D18: BZT52C9V1-7-F, Diode_SMD:D_SOD-123, F.Cu at (96.6, 119.0)
- added D18: BZT52C9V1-7-F, Diode_SMD:D_SOD-123, F.Cu at (65.8, 119.0)
- added D18: BZT52C9V1-7-F, Diode_SMD:D_SOD-123, F.Cu at (50.4, 119.0)
- added J10: Conn_01x06_Socket, Connector_PinSocket_2.54mm:PinSocket_2x03_P2.54mm_Vertical, F.Cu at (90.2, 130.0)
- added J10: Conn_01x06_Socket, Connector_PinSocket_2.54mm:PinSocket_2x03_P2.54mm_Vertical, F.Cu at (44.0, 130.0)
- added J10: Conn_01x06_Socket, Connector_PinSocket_2.54mm:PinSocket_2x03_P2.54mm_Vertical, F.Cu at (59.4, 130.0)
- added J3: Conn_01x06_Socket, Connector_PinSocket_2.54mm:PinSocket_2x03_P2.54mm_Vertical, F.Cu at (44.0, 105.9)
- added J3: Conn_01x06_Socket, Connector_PinSocket_2.54mm:PinSocket_2x03_P2.54mm_Vertical, F.Cu at (90.2, 105.9)
- added J3: Conn_01x06_Socket, Connector_PinSocket_2.54mm:PinSocket_2x03_P2.54mm_Vertical, F.Cu at (59.4, 105.9)
- added Q25: NMOS, Package_TO_SOT_SMD:SOT-89-3, F.Cu at (56.7, 88.9)
- added Q25: NMOS, Package_TO_SOT_SMD:SOT-89-3, F.Cu at (41.3, 89.0)
- added Q25: NMOS, Package_TO_SOT_SMD:SOT-89-3, F.Cu at (87.5, 89.0)
- added Q26: NMOS, Package_TO_SOT_SMD:SOT-89-3, F.Cu at (61.9, 89.0)
- added Q26: NMOS, Package_TO_SOT_SMD:SOT-89-3, F.Cu at (92.7, 89.0)
- added Q26: NMOS, Package_TO_SOT_SMD:SOT-89-3, F.Cu at (46.5, 89.0)
- added Q27: NMOS, Package_TO_SOT_SMD:SOT-89-3, F.Cu at (51.6, 88.9)
- added Q27: NMOS, Package_TO_SOT_SMD:SOT-89-3, F.Cu at (97.8, 88.9)
- added Q27: NMOS, Package_TO_SOT_SMD:SOT-89-3, F.Cu at (67.0, 88.9)
- added Q28: PMOS, Package_TO_SOT_SMD:SOT-89-3, F.Cu at (56.7, 101.1)
- added Q28: PMOS, Package_TO_SOT_SMD:SOT-89-3, F.Cu at (41.3, 101.1)
- added Q28: PMOS, Package_TO_SOT_SMD:SOT-89-3, F.Cu at (87.5, 101.1)
- added Q29: PMOS, Package_TO_SOT_SMD:SOT-89-3, F.Cu at (61.9, 101.1)
- added Q29: PMOS, Package_TO_SOT_SMD:SOT-89-3, F.Cu at (92.7, 101.1)
- added Q29: PMOS, Package_TO_SOT_SMD:SOT-89-3, F.Cu at (46.5, 101.1)
- added Q30: PMOS, Package_TO_SOT_SMD:SOT-89-3, F.Cu at (67.0, 101.1)
- added Q30: PMOS, Package_TO_SOT_SMD:SOT-89-3, F.Cu at (97.8, 101.1)
- added Q30: PMOS, Package_TO_SOT_SMD:SOT-89-3, F.Cu at (51.6, 101.1)
- added Q31: NMOS, Package_TO_SOT_SMD:SOT-89-3, F.Cu at (87.7, 125.5)
- added Q31: NMOS, Package_TO_SOT_SMD:SOT-89-3, F.Cu at (56.9, 125.5)
- added Q31: NMOS, Package_TO_SOT_SMD:SOT-89-3, F.Cu at (41.5, 125.5)
- added Q32: NMOS, Package_TO_SOT_SMD:SOT-89-3, F.Cu at (62.0, 125.4)
- added Q32: NMOS, Package_TO_SOT_SMD:SOT-89-3, F.Cu at (92.8, 125.4)
- added Q32: NMOS, Package_TO_SOT_SMD:SOT-89-3, F.Cu at (46.6, 125.4)
- added Q33: NMOS, Package_TO_SOT_SMD:SOT-89-3, F.Cu at (51.8, 125.4)
- added Q33: NMOS, Package_TO_SOT_SMD:SOT-89-3, F.Cu at (98.0, 125.4)
- added Q33: NMOS, Package_TO_SOT_SMD:SOT-89-3, F.Cu at (67.2, 125.4)
- added Q34: PMOS, Package_TO_SOT_SMD:SOT-89-3, F.Cu at (57.0, 113.0)
- added Q34: PMOS, Package_TO_SOT_SMD:SOT-89-3, F.Cu at (87.8, 113.0)
- added Q34: PMOS, Package_TO_SOT_SMD:SOT-89-3, F.Cu at (41.6, 113.0)
- added Q35: PMOS, Package_TO_SOT_SMD:SOT-89-3, F.Cu at (46.7, 113.0)
- added Q35: PMOS, Package_TO_SOT_SMD:SOT-89-3, F.Cu at (92.9, 113.0)
- added Q35: PMOS, Package_TO_SOT_SMD:SOT-89-3, F.Cu at (62.1, 113.0)
- added Q36: PMOS, Package_TO_SOT_SMD:SOT-89-3, F.Cu at (51.9, 113.0)
- added Q36: PMOS, Package_TO_SOT_SMD:SOT-89-3, F.Cu at (67.3, 113.0)
- added Q36: PMOS, Package_TO_SOT_SMD:SOT-89-3, F.Cu at (98.1, 113.0)
- added R25: 10M, Resistor_SMD:R_0603_1608Metric, F.Cu at (85.8, 93.4)
- added R26: 10M, Resistor_SMD:R_0603_1608Metric, F.Cu at (44.7, 93.5)
- added R26: 10M, Resistor_SMD:R_0603_1608Metric, F.Cu at (90.9, 93.5)
- added R26: 10M, Resistor_SMD:R_0603_1608Metric, F.Cu at (60.1, 93.5)
- added R27: 10M, Resistor_SMD:R_0603_1608Metric, F.Cu at (96.0, 93.4)
- added R27: 10M, Resistor_SMD:R_0603_1608Metric, F.Cu at (49.8, 93.4)
- added R27: 10M, Resistor_SMD:R_0603_1608Metric, F.Cu at (65.2, 93.4)
- added R28: 10K, Resistor_SMD:R_0603_1608Metric, F.Cu at (40.6, 96.6)
- added R28: 10K, Resistor_SMD:R_0603_1608Metric, F.Cu at (86.8, 96.6)
- added R28: 10K, Resistor_SMD:R_0603_1608Metric, F.Cu at (56.0, 96.6)
- added R29: 10K, Resistor_SMD:R_0603_1608Metric, F.Cu at (92.0, 96.7)
- added R29: 10K, Resistor_SMD:R_0603_1608Metric, F.Cu at (61.2, 96.7)
- added R29: 10K, Resistor_SMD:R_0603_1608Metric, F.Cu at (45.8, 96.7)
- added R30: 10K, Resistor_SMD:R_0603_1608Metric, F.Cu at (66.3, 96.7)
- added R30: 10K, Resistor_SMD:R_0603_1608Metric, F.Cu at (50.9, 96.7)
- added R30: 10K, Resistor_SMD:R_0603_1608Metric, F.Cu at (97.1, 96.7)
- added R31: 10M, Resistor_SMD:R_0603_1608Metric, F.Cu at (58.7, 120.9)
- added R31: 10M, Resistor_SMD:R_0603_1608Metric, F.Cu at (43.2, 120.9)
- added R31: 10M, Resistor_SMD:R_0603_1608Metric, F.Cu at (89.4, 120.9)
- added R32: 10M, Resistor_SMD:R_0603_1608Metric, F.Cu at (63.8, 120.6)
- added R32: 10M, Resistor_SMD:R_0603_1608Metric, F.Cu at (94.6, 120.6)
- added R32: 10M, Resistor_SMD:R_0603_1608Metric, F.Cu at (48.4, 120.6)
- added R33: 10M, Resistor_SMD:R_0603_1608Metric, F.Cu at (68.9, 120.6)
- added R33: 10M, Resistor_SMD:R_0603_1608Metric, F.Cu at (53.5, 120.6)
- added R33: 10M, Resistor_SMD:R_0603_1608Metric, F.Cu at (99.7, 120.6)
- added R34: 10K, Resistor_SMD:R_0603_1608Metric, F.Cu at (57.9, 117.6)
- added R34: 10K, Resistor_SMD:R_0603_1608Metric, F.Cu at (42.4, 117.6)
- added R34: 10K, Resistor_SMD:R_0603_1608Metric, F.Cu at (88.6, 117.6)
- added R35: 10K, Resistor_SMD:R_0603_1608Metric, F.Cu at (93.7, 117.5)
- added R35: 10K, Resistor_SMD:R_0603_1608Metric, F.Cu at (62.9, 117.5)
- added R35: 10K, Resistor_SMD:R_0603_1608Metric, F.Cu at (47.5, 117.5)
- added R36: 10K, Resistor_SMD:R_0603_1608Metric, F.Cu at (67.9, 117.5)
- added R36: 10K, Resistor_SMD:R_0603_1608Metric, F.Cu at (52.5, 117.5)
- added R36: 10K, Resistor_SMD:R_0603_1608Metric, F.Cu at (98.7, 117.5)
- D1, D10, D11, D12, D13, D14, D15, D16, D17, D18, D19, D2, D20, D21, D22, D23, D24, D3, D4, D5, D6, D7, D8, D9: value 1N47xxA -> BZT52C9V1-7-F; footprint Diode_THT:D_DO-41_SOD81_P10.16mm_Horizontal -> Diode_SMD:D_SOD-123
- Q1, Q10, Q11, Q12, Q13, Q14, Q15, Q16, Q17, Q18, Q19, Q2, Q20, Q21, Q22, Q23, Q24, Q25, Q26, Q27, Q28, Q29, Q3, Q30, Q31, Q32, Q33, Q34, Q35, Q36, Q37, Q38, Q39, Q4, Q40, Q41, Q42, Q43, Q44, Q45, Q46, Q47, Q48, Q5, Q6, Q7, Q8, Q9: footprint Package_TO_SOT_THT:TO-92_Inline -> Package_TO_SOT_SMD:SOT-89-3
- R1, R10, R11, R12, R13, R14, R15, R16, R17, R18, R19, R2, R20, R21, R22, R23, R24, R25, R26, R27, R28, R29, R3, R30, R31, R32, R33, R34, R35, R36, R37, R38, R39, R4, R40, R41, R42, R43, R44, R45, R46, R47, R48, R5, R6, R7, R8, R9: footprint Resistor_THT:R_Axial_DIN0207_L6.3mm_D2.5mm_P7.62mm_Horizontal -> Resistor_SMD:R_0603_1608Metric
- R49: footprint Resistor_THT:R_Axial_DIN0207_L6.3mm_D2.5mm_P7.62mm_Horizontal -> Resistor_SMD:R_0603_1608Metric; moved to B.Cu
- moved U4 125.7 mm to (43.5, 69.2)
- moved J7 125.6 mm to (42.2, 79.6)
- moved R49 122.4 mm to (42.3, 75.5), turned to -90 degrees
- moved J5 107.8 mm to (42.0, 58.7)
- moved D19 99.8 mm to (204.2, 133.2)
- moved D20 99.8 mm to (204.2, 137.4)
- moved D21 99.8 mm to (204.2, 141.7)
- moved D22 99.8 mm to (204.2, 145.9)
- moved D23 99.8 mm to (204.2, 150.2)
- moved D24 99.8 mm to (204.2, 154.4)
- moved Q37 99.8 mm to (204.3, 116.9)
- moved Q40 99.8 mm to (210.8, 116.9)
- moved Q43 99.8 mm to (217.3, 116.9)
- moved Q46 99.8 mm to (223.8, 116.9)
- moved R39 99.8 mm to (193.1, 123.8)
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Routing:
- net Net-(D16-A): track 0.00 -> 35.2 mm
- net /DotDriver2/+450V: track 0.00 -> 15.3 mm
- net Net-(Q31-D): track 0.00 -> 7.58 mm

Commit message: placement done
Parts:
- removed the D13 at (58.1, 94.8)
- removed the D13 at (88.9, 94.8)
- removed the D13 at (42.7, 94.8)
- removed the D14 at (78.6, 95.0)
- removed the D14 at (63.2, 95.0)
- removed the D14 at (47.8, 95.0)
- removed the D15 at (83.8, 95.0)
- removed the D15 at (99.2, 95.0)
- removed the D15 at (53.0, 95.0)
- removed the D16 at (86.4, 118.9)
- removed the D16 at (55.7, 118.9)
- removed the D16 at (71.0, 118.9)
- removed the D17 at (45.4, 118.9)
- removed the D17 at (76.2, 118.9)
- removed the D17 at (91.6, 118.9)
- removed the D18 at (96.6, 119.0)
- removed the D18 at (65.8, 119.0)
- removed the D18 at (50.4, 119.0)
- removed the J10 at (90.2, 130.0)
- removed the J10 at (44.0, 130.0)
- removed the J10 at (59.4, 130.0)
- removed the J3 at (74.8, 105.9)
- removed the J3 at (44.0, 105.9)
- removed the J3 at (90.2, 105.9)
- removed the Q25 at (56.7, 88.9)
- removed the Q25 at (41.3, 89.0)
- removed the Q25 at (87.5, 89.0)
- removed the Q26 at (61.9, 89.0)
- removed the Q26 at (77.2, 89.0)
- removed the Q26 at (46.5, 89.0)
- removed the Q27 at (51.6, 88.9)
- removed the Q27 at (82.4, 88.9)
- removed the Q27 at (97.8, 88.9)
- removed the Q28 at (56.7, 101.1)
- removed the Q28 at (41.3, 101.1)
- removed the Q28 at (87.5, 101.1)
- removed the Q29 at (61.9, 101.1)
- removed the Q29 at (46.5, 101.1)
- removed the Q29 at (77.2, 101.1)
- removed the Q30 at (97.8, 101.1)
- removed the Q30 at (51.6, 101.1)
- removed the Q30 at (82.4, 101.1)
- removed the Q31 at (87.7, 125.5)
- removed the Q31 at (56.9, 125.5)
- removed the Q31 at (72.2, 125.5)
- removed the Q32 at (77.4, 125.4)
- removed the Q32 at (92.8, 125.4)
- removed the Q32 at (46.6, 125.4)
- removed the Q33 at (51.8, 125.4)
- removed the Q33 at (98.0, 125.4)
- removed the Q33 at (67.2, 125.4)
- removed the Q34 at (57.0, 113.0)
- removed the Q34 at (87.8, 113.0)
- removed the Q34 at (72.4, 113.0)
- removed the Q35 at (46.7, 113.0)
- removed the Q35 at (92.9, 113.0)
- removed the Q35 at (77.5, 113.0)
- removed the Q36 at (51.9, 113.0)
- removed the Q36 at (67.3, 113.0)
- removed the Q36 at (98.1, 113.0)
- removed the R25 at (85.8, 93.4)
- removed the R26 at (75.5, 93.5)
- removed the R26 at (44.7, 93.5)
- removed the R26 at (60.1, 93.5)
- removed the R27 at (96.0, 93.4)
- removed the R27 at (49.8, 93.4)
- removed the R27 at (80.6, 93.4)
- removed the R28 at (40.6, 96.6)
- removed the R28 at (86.8, 96.6)
- removed the R28 at (56.0, 96.6)
- removed the R29 at (76.5, 96.7)
- removed the R29 at (61.2, 96.7)
- removed the R29 at (45.8, 96.7)
- removed the R30 at (50.9, 96.7)
- removed the R30 at (97.1, 96.7)
- removed the R30 at (81.7, 96.7)
- removed the R31 at (58.7, 120.9)
- removed the R31 at (89.4, 120.9)
- removed the R31 at (74.0, 120.9)
- removed the R32 at (94.6, 120.6)
- removed the R32 at (79.2, 120.6)
- removed the R32 at (48.4, 120.6)
- removed the R33 at (68.9, 120.6)
- removed the R33 at (53.5, 120.6)
- removed the R33 at (99.7, 120.6)
- removed the R34 at (73.2, 117.6)
- removed the R34 at (57.9, 117.6)
- removed the R34 at (88.6, 117.6)
- removed the R35 at (78.2, 117.5)
- removed the R35 at (93.7, 117.5)
- removed the R35 at (47.5, 117.5)
- removed the R36 at (67.9, 117.5)
- removed the R36 at (52.5, 117.5)
- removed the R36 at (98.7, 117.5)
- U1, U2, U3: footprint Package_DIP:DIP-16_W7.62mm -> Package_SO:SOIC-16W_5.3x10.2mm_P1.27mm
- moved J1 235.9 mm to (45.0, 130.0), turned to 90 degrees
- moved J9 217.9 mm to (60.0, 130.0), turned to 90 degrees
- moved Q19 190.1 mm to (57.3, 125.1), turned to -90 degrees
- moved Q22 189.2 mm to (57.2, 112.6), turned to 90 degrees
- moved Q20 182.7 mm to (62.4, 125.1), turned to -90 degrees
- moved Q23 182.0 mm to (62.4, 112.7), turned to 90 degrees
- moved J11 181.2 mm to (90.0, 130.0), turned to 90 degrees
- moved Q21 175.2 mm to (67.5, 125.1), turned to -90 degrees
- moved Q24 174.7 mm to (67.5, 112.7), turned to 90 degrees
- moved J0 174.1 mm to (60.0, 105.9), turned to 90 degrees
- moved Q13 172.6 mm to (57.2, 101.8), turned to -90 degrees
- moved Q17 165.4 mm to (62.4, 101.8), turned to -90 degrees
- moved Q3 161.2 mm to (57.2, 89.3), turned to 90 degrees
- moved D10 160.1 mm to (58.5, 118.6), turned to -90 degrees
- moved D4 158.2 mm to (55.9, 95.3), turned to 90 degrees
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Connections:
- J7 pad 1: DOUT -> DIN
- J7 pad 2: SRCLK -> SRCLK_IN
- J7 pad 3: RCLK -> RCLK_IN
- J7 pad 4: OE -> OE_IN
- J8 pad 1: DIN -> DOUT
- J8 pad 2: SRCLK_IN -> SRCLK
- J8 pad 3: RCLK_IN -> RCLK
- J8 pad 4: OE_IN -> OE
Routing:
- net Net-(D16-A): track 35.2 -> 0.00 mm
- net /DotDriver2/+450V: track 15.3 -> 0.00 mm
- net Net-(Q31-D): track 7.58 -> 0.00 mm
Other:
- board outline added: 62 x 73.3 mm

Commit message: initial layout of dev
Parts:
- moved R49 12.2 mm to (54.2, 73.0), turned to 90 degrees
- moved J6 6.07 mm to (81.4, 66.5)
- moved J5 1.27 mm to (59.1, 66.2), turned to 180 degrees
- moved D9 0.46 mm to (66.2, 95.5)
- moved R7 0.31 mm to (58.3, 94.2)
- moved R12 0.29 mm to (68.2, 94.1)
- moved R8 0.27 mm to (63.2, 94.0)
Connections:
- D1 pad 1: /DotDriver/+450V -> +450V
- D10 pad 1: /DotDriver1/+450V -> +450V
- D11 pad 1: /DotDriver1/+450V -> +450V
- D12 pad 1: /DotDriver1/+450V -> +450V
- D13 pad 1: /DotDriver2/+450V -> +450V
- D14 pad 1: /DotDriver2/+450V -> +450V
- D15 pad 1: /DotDriver2/+450V -> +450V
- D16 pad 1: /DotDriver2/+450V -> +450V
- D17 pad 1: /DotDriver2/+450V -> +450V
- D18 pad 1: /DotDriver2/+450V -> +450V
- D19 pad 1: /DotDriver3/+450V -> +450V
- D2 pad 1: /DotDriver/+450V -> +450V
- D20 pad 1: /DotDriver3/+450V -> +450V
- D21 pad 1: /DotDriver3/+450V -> +450V
- D22 pad 1: /DotDriver3/+450V -> +450V
- D23 pad 1: /DotDriver3/+450V -> +450V
- D24 pad 1: /DotDriver3/+450V -> +450V
- D3 pad 1: /DotDriver/+450V -> +450V
- D4 pad 1: /DotDriver1/+450V -> +450V
- D5 pad 1: /DotDriver/+450V -> +450V
- D6 pad 1: /DotDriver/+450V -> +450V
- D7 pad 1: /DotDriver/+450V -> +450V
- D8 pad 1: /DotDriver1/+450V -> +450V
- D9 pad 1: /DotDriver1/+450V -> +450V
- J5 pad 2: /+450V -> +450V
- J6 pad 2: /+450V -> +450V
- Q13 pad 1: /DotDriver1/+450V -> +450V
- Q14 pad 1: /DotDriver/+450V -> +450V
- Q15 pad 1: /DotDriver/+450V -> +450V
- Q16 pad 1: /DotDriver/+450V -> +450V
- Q17 pad 1: /DotDriver1/+450V -> +450V
- Q18 pad 1: /DotDriver1/+450V -> +450V
- Q2 pad 1: /DotDriver/+450V -> +450V
- Q22 pad 1: /DotDriver1/+450V -> +450V
- Q23 pad 1: /DotDriver1/+450V -> +450V
- Q24 pad 1: /DotDriver1/+450V -> +450V
- Q28 pad 1: /DotDriver2/+450V -> +450V
- Q29 pad 1: /DotDriver2/+450V -> +450V
- Q30 pad 1: /DotDriver2/+450V -> +450V
- Q34 pad 1: /DotDriver2/+450V -> +450V
- Q35 pad 1: /DotDriver2/+450V -> +450V
- Q36 pad 1: /DotDriver2/+450V -> +450V
- Q40 pad 1: /DotDriver3/+450V -> +450V
- Q41 pad 1: /DotDriver3/+450V -> +450V
- Q42 pad 1: /DotDriver3/+450V -> +450V
- Q46 pad 1: /DotDriver3/+450V -> +450V
- Q47 pad 1: /DotDriver3/+450V -> +450V
- Q48 pad 1: /DotDriver3/+450V -> +450V
- Q5 pad 1: /DotDriver/+450V -> +450V
- Q7 pad 1: /DotDriver/+450V -> +450V
- R1 pad 1: /DotDriver/+450V -> +450V
- R13 pad 1: /DotDriver/+450V -> +450V
- R14 pad 1: /DotDriver/+450V -> +450V
- R15 pad 1: /DotDriver/+450V -> +450V
- R16 pad 1: /DotDriver1/+450V -> +450V
- R17 pad 1: /DotDriver1/+450V -> +450V
- R18 pad 1: /DotDriver1/+450V -> +450V
- R22 pad 1: /DotDriver1/+450V -> +450V
- R23 pad 1: /DotDriver1/+450V -> +450V
- R24 pad 1: /DotDriver1/+450V -> +450V
- R28 pad 1: /DotDriver2/+450V -> +450V
- R29 pad 1: /DotDriver2/+450V -> +450V
- R30 pad 1: /DotDriver2/+450V -> +450V
- R34 pad 1: /DotDriver2/+450V -> +450V
- R35 pad 1: /DotDriver2/+450V -> +450V
- R36 pad 1: /DotDriver2/+450V -> +450V
- R4 pad 1: /DotDriver/+450V -> +450V
- R40 pad 1: /DotDriver3/+450V -> +450V
- R41 pad 1: /DotDriver3/+450V -> +450V
- R42 pad 1: /DotDriver3/+450V -> +450V
- R46 pad 1: /DotDriver3/+450V -> +450V
- R47 pad 1: /DotDriver3/+450V -> +450V
- R48 pad 1: /DotDriver3/+450V -> +450V
- R6 pad 1: /DotDriver/+450V -> +450V
Routing:
- net +450V: track 0.00 -> 229.3 mm
- net +5V: track 0.00 -> 89.3 mm, vias 0 -> 4
- net SRCLK: track 0.00 -> 65.8 mm, vias 0 -> 4
- net RCLK: track 0.00 -> 51.8 mm, vias 0 -> 4
- net OE: track 0.00 -> 51.1 mm, vias 0 -> 1
- net /DotDriver/UP2: track 0.00 -> 50.5 mm, vias 0 -> 2
- net /DotDriver3/UP6: track 0.00 -> 48.8 mm, vias 0 -> 2
- net /DotDriver/UP4: track 0.00 -> 48.0 mm, vias 0 -> 2
- net /DotDriver3/UP4: track 0.00 -> 47.6 mm, vias 0 -> 2
- net /DotDriver/UP6: track 0.00 -> 47.2 mm, vias 0 -> 2
- net /DotDriver2/UP4: track 0.00 -> 47.1 mm, vias 0 -> 2
- net /DotDriver1/UP2: track 0.00 -> 46.5 mm, vias 0 -> 2
- net /DotDriver1/UP4: track 0.00 -> 45.6 mm, vias 0 -> 2
- net /DotDriver3/UP2: track 0.00 -> 45.2 mm, vias 0 -> 2
- net /DotDriver2/UP6: track 0.00 -> 44.9 mm, vias 0 -> 2
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- added copper zone on B.Cu, net +450V
- added copper zone on B.Cu, net GND
- added copper zone on F.Cu, net GND

Commit message: layout finished
Parts:
- added R50: 1K, Resistor_SMD:R_0603_1608Metric, B.Cu at (42.5, 89.2)
- added R51: 1K, Resistor_SMD:R_0603_1608Metric, B.Cu at (57.2, 89.8)
- added R52: 1K, Resistor_SMD:R_0603_1608Metric, B.Cu at (72.8, 89.8)
- added R53: 1K, Resistor_SMD:R_0603_1608Metric, B.Cu at (88.0, 90.5)
- added R54: 1K, Resistor_SMD:R_0603_1608Metric, B.Cu at (47.0, 89.2)
- added R55: 1K, Resistor_SMD:R_0603_1608Metric, B.Cu at (62.5, 90.0)
- added R56: 1K, Resistor_SMD:R_0603_1608Metric, B.Cu at (77.8, 89.8)
- added R57: 1K, Resistor_SMD:R_0603_1608Metric, B.Cu at (92.5, 90.3)
- added R58: 1K, Resistor_SMD:R_0603_1608Metric, B.Cu at (52.8, 90.2)
- added R59: 1K, Resistor_SMD:R_0603_1608Metric, B.Cu at (68.2, 89.5)
- added R60: 1K, Resistor_SMD:R_0603_1608Metric, B.Cu at (82.8, 90.0)
- added R61: 1K, Resistor_SMD:R_0603_1608Metric, B.Cu at (98.2, 90.5)
- added R62: 1K, Resistor_SMD:R_0603_1608Metric, B.Cu at (41.8, 126.8)
- added R63: 1K, Resistor_SMD:R_0603_1608Metric, B.Cu at (57.2, 126.8)
- added R64: 1K, Resistor_SMD:R_0603_1608Metric, B.Cu at (72.5, 126.8)
- added R65: 1K, Resistor_SMD:R_0603_1608Metric, B.Cu at (88.0, 126.8)
- added R66: 1K, Resistor_SMD:R_0603_1608Metric, B.Cu at (47.0, 126.8)
- added R67: 1K, Resistor_SMD:R_0603_1608Metric, B.Cu at (62.5, 126.8)
- added R68: 1K, Resistor_SMD:R_0603_1608Metric, B.Cu at (77.8, 126.8)
- added R69: 1K, Resistor_SMD:R_0603_1608Metric, B.Cu at (93.0, 126.8)
- added R70: 1K, Resistor_SMD:R_0603_1608Metric, B.Cu at (52.2, 126.8)
- added R71: 1K, Resistor_SMD:R_0603_1608Metric, B.Cu at (67.5, 126.8)
- added R72: 1K, Resistor_SMD:R_0603_1608Metric, B.Cu at (83.0, 126.8)
- added R73: 1K, Resistor_SMD:R_0603_1608Metric, B.Cu at (98.2, 126.8)
Routing:
- net +450V: track 229.3 -> 284.1 mm, vias 0 -> 2
- net /DotDriver1/UP4: track 45.6 -> 48.3 mm
- net /DotDriver2/UP2: track 44.1 -> 46.8 mm
- net /DotDriver2/UP4: track 47.1 -> 49.9 mm
- net /DotDriver1/UP6: track 44.3 -> 47.1 mm
- net /DotDriver1/UP2: track 46.5 -> 49.3 mm
- net /DotDriver/UP6: track 47.2 -> 49.9 mm
- net /DotDriver2/UP6: track 44.9 -> 47.6 mm
- net /DotDriver3/UP4: track 47.6 -> 50.3 mm
- net /DotDriver3/UP6: track 48.8 -> 51.5 mm
- net /DotDriver3/UP2: track 45.2 -> 47.8 mm
- net /DotDriver3/UP5: vias 0 -> 1
- net /DotDriver3/UP3: vias 0 -> 1
- net /DotDriver3/UP1: vias 0 -> 1
- net /DotDriver2/UP5: vias 0 -> 1
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Other:
- board text added: "Charles Van Hook Leah Jones"

Commit message: led board
Parts:
- moved J1 3.00 mm to (45.0, 133.0)
- moved J10 3.00 mm to (75.0, 133.0)
- moved J11 3.00 mm to (90.0, 133.0)
- moved J9 3.00 mm to (60.0, 133.0)
Other:
- board size 62 x 73.3 mm -> 62 x 80.2 mm
Changed lines of the file:
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@@
 	(footprint "Connector_PinSocket_2.54mm:PinSocket_2x03_P2.54mm_Vertical"
 		(layer "F.Cu")
-		(at 90 130 90)
+		(at 90 133 90)
 		(descr "Through hole straight socket strip, 2x03, 2.54mm pitch, double cols (from Kicad 4.0.7), script generated")
 		(tags "Through hole socket strip THT 2x03 2.54mm double row")
@@
 	(footprint "Connector_PinSocket_2.54mm:PinSocket_2x03_P2.54mm_Vertical"
 		(layer "F.Cu")
-		(at 60 130 90)
+		(at 60 133 90)
 		(descr "Through hole straight socket strip, 2x03, 2.54mm pitch, double cols (from Kicad 4.0.7), script generated")
 		(tags "Through hole socket strip THT 2x03 2.54mm double row")
@@
 	(footprint "Connector_PinSocket_2.54mm:PinSocket_2x03_P2.54mm_Vertical"
 		(layer "F.Cu")
-		(at 75 130 90)
+		(at 75 133 90)
 		(descr "Through hole straight socket strip, 2x03, 2.54mm pitch, double cols (from Kicad 4.0.7), script generated")
 		(tags "Through hole socket strip THT 2x03 2.54mm double row")
@@
 	(footprint "Connector_PinSocket_2.54mm:PinSocket_2x03_P2.54mm_Vertical"
 		(layer "F.Cu")
-		(at 45 130 90)
+		(at 45 133 90)
 		(descr "Through hole straight socket strip, 2x03, 2.54mm pitch, double cols (from Kicad 4.0.7), script generated")
 		(tags "Through hole socket strip THT 2x03 2.54mm double row")
@@
 	)
 	(gr_arc
-		(start 41.05 134.8)
-		(mid 39.635786 134.214214)
-		(end 39.05 132.8)
+		(start 41.05 141.75)
+		(mid 39.635786 141.164214)
+		(end 39.05 139.75)
 		(stroke
 			(width 0.2)
@@
 	)
 	(gr_line
-		(start 39.05 132.8)
+		(start 39.05 139.75)
 		(end 39.05 63.5)
 		(stroke
@@
 	(gr_line
 		(start 101 63.5)
-		(end 101 132.8)
+		(end 101 139.75)
 		(stroke
 			(width 0.2)
@@
 	)
 	(gr_arc
-		(start 101 132.8)
-		(mid 100.414214 134.214214)
-		(end 99 134.8)
+		(start 101 139.75)
+		(mid 100.414214 141.164214)
+		(end 99 141.75)
 		(stroke
 			(width 0.2)
@@
 	)
 	(gr_line
-		(start 99 134.8)
-		(end 41.05 134.8)
+		(start 99 141.75)
+		(end 41.05 141.75)
 		(stroke
 			(width 0.2)
@@
 	)
 	(via
-		(at 98.5 132.25)
-		(size 4)
-		(drill 2.5)
+		(at 98.490699 139.25)
+		(size 5.5)
+		(drill 3)
 		(layers "F.Cu" "B.Cu")
 		(free yes)
@@
 	(via
 		(at 98.5 64.042327)
-		(size 4)
-		(drill 2.5)
+		(size 5.5)
+		(drill 3)
 		(layers "F.Cu" "B.Cu")
 		(free yes)
@@
 	)
 	(via
-		(at 41.55 132.3)
-		(size 4)
-		(drill 2.5)
+		(at 41.487835 139.195946)
+		(size 5.5)
+		(drill 3)
 		(layers "F.Cu" "B.Cu")
 		(free yes)
@@
 	(via
 		(at 41.55 64)
-		(size 4)
-		(drill 2.5)
+		(size 5.5)
+		(drill 3)
 		(layers "F.Cu" "B.Cu")
 		(free yes)
@@
 		(min_thickness 0.25)
 		(filled_areas_thickness no)
-		(fill yes
+		(fill
 			(thermal_gap 0.5)
 			(thermal_bridge_width 0.5)
@@
 		(polygon
 			(pts
-				(xy 38 59.25) (xy 38.25 135.5) (xy 103.25 135.5) (xy 103.25 59.75) (xy 103.5 58.75) (xy 38 59)
+				(xy 38 59.25) (xy 38.281967 145.25) (xy 103.25 145.25) (xy 103.25 59.75) (xy 103.5 58.75) (xy 38 59)
 			)
 		)
